File: z3660-board/Z3660_kicad/Z3660_v021a.kicad_pcb (KiCad board)
At the start: 4 copper layers, 173.9 x 92.8 mm, 178 parts, among them CN1 KEL-8817-200-170S-F, CN2 Conn_02x40_Odd_Even, CN3 Conn_02x40_Odd_Even, J1 Jumper_2_Open, J2 Conn_02x07_Odd_Even, U1 LTC2990, U10 74FCT543A, U11 74FCT543A, U12 74FCT543A, U13 74FCT543A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

Commit message: Update led values values to differentiate green and red.
Parts:
- D1: value LED_Small -> LED_Small_Green
- D2: value LED_Small -> LED_Small_Red
Changed lines of the file:
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@@
     (title "Z3660 by sHaNsHe (Double H Tech)")
     (date "2023-08-06")
-    (rev "v0.21")
+    (rev "v0.21a")
+    (comment 1 "v0.21a Changed Array Networks")
   )
   (layers
@@
         (effects (font (size 1 1) (thickness 0.15)))
     )
-    (fp_text value "LED_Small" (at 0 1.82 180) (layer "F.Fab")
+    (fp_text value "LED_Small_Green" (at 0 1.82 180) (layer "F.Fab")
         (effects (font (size 1 1) (thickness 0.15)))
     )
@@
         (effects (font (size 1 1) (thickness 0.15)))
     )
-    (fp_text value "LED_Small" (at 0 1.82 180) (layer "F.Fab")
+    (fp_text value "LED_Small_Red" (at 0 1.82 180) (layer "F.Fab")
         (effects (font (size 1 1) (thickness 0.15)))
     )
