File: z3660-board/Z3660_kicad/Sheet2.kicad_sch (KiCad schematic)
At the start: 19 parts, among them U10 74FCT543A, U11 74FCT543A, U12 74FCT543A, U13 74FCT543A, U14 74FCT543A, U6 74FCT543A, U7 74FCT543A, U8 74FCT543A, U9 74FCT543A

Commit message: Update to version v0.21a
Parts:
- C29, C30, C31, C32, C33, C34, C35, C36, C37: footprint Capacitor_SMD:C_0805_2012Metric_Pad1.18x1.45mm_HandSolder -> Z3660_v02:C_0805_2012Metric_Pad1.18x1.45mm_HandSolder
- R14: footprint Resistor_SMD:R_0805_2012Metric_Pad1.20x1.40mm_HandSolder -> Z3660_v02:R_0805_2012Metric_Pad1.20x1.40mm_HandSolder
- U10, U11, U12, U13, U14, U6, U7, U8, U9: footprint Package_SO:SOIC-24W_7.5x15.4mm_P1.27mm -> Z3660_v02:SOIC-24W_7.5x15.4mm_P1.27mm
