File: z3660-board/Z3660_kicad/Sheet3.kicad_sch (KiCad schematic)
At the start: 28 parts, among them J1 Jumper_2_Open, J2 Conn_02x07_Odd_Even, U1A1 RH5VA43A, U1B1 BU4942, U2 XC95144XL-TQ144, U3 SN74CB3T3245PW

Commit message: Update to version v0.21a
Parts:
- C1, C10, C2, C3, C4, C5, C6, C7, C8, C9: footprint Capacitor_SMD:C_0805_2012Metric_Pad1.18x1.45mm_HandSolder -> Z3660_v02:C_0805_2012Metric_Pad1.18x1.45mm_HandSolder
- C400A1: footprint Capacitor_SMD:C_1812_4532Metric_Pad1.57x3.40mm_HandSolder -> Z3660_v02:C_1812_4532Metric_Pad1.57x3.40mm_HandSolder
- J1: footprint Connector_PinHeader_2.54mm:PinHeader_1x02_P2.54mm_Vertical -> Z3660_v02:PinHeader_1x02_P2.54mm_Vertical
- J2: footprint Connector_IDC:IDC-Header_2x07_P2.54mm_Vertical -> Z3660_v02:IDC-Header_2x07_P2.54mm_Vertical
- JP8: footprint Jumper:SolderJumper-3_P1.3mm_Bridged12_RoundedPad1.0x1.5mm_NumberLabels -> Z3660_v02:SolderJumper-3_P1.3mm_Bridged12_RoundedPad1.0x1.5mm_NumberLabels
- R1, R2, R28, R29, R3, R4: footprint Resistor_SMD:R_0805_2012Metric_Pad1.20x1.40mm_HandSolder -> Z3660_v02:R_0805_2012Metric_Pad1.20x1.40mm_HandSolder
- TP9: footprint TestPoint:TestPoint_THTPad_2.0x2.0mm_Drill1.0mm -> Z3660_v02:TestPoint_THTPad_2.0x2.0mm_Drill1.0mm
- U1B1: footprint Package_SO:TSOP-5_1.65x3.05mm_P0.95mm -> Z3660_v02:TSOP-5_1.65x3.05mm_P0.95mm
