File: z3660-board/Z3660_kicad/Sheet4.kicad_sch (KiCad schematic)
At the start: 9 parts, among them CN1 KEL-8817-200-170S-F

Commit message: Update to version v0.21a
Parts:
- removed RN10, RN11, RN12, RN7, RN8, RN9: 1k, Z3660_v02:R_Array_Convex_8x0602, symbol Z3660_v02:R_Pack08
- added RN1 (x12): 1k, Z3660_v02:R_Array_Convex_4x0603, symbol Z3660_v02:R_Pack04
Connections:
- net +3V3: now also RN1.1 (R1.1), RN1.1 (R1.1), RN1.1 (R1.1), RN1.1 (R1.1), RN1.1 (R1.1), RN1.1 (R1.1), RN1.1 (R1.1), RN1.1 (R1.1), RN1.1 (R1.1), RN1.1 (R1.1), RN1.1 (R1.1), RN1.1 (R1.1), RN1.2 (R2.1), RN1.2 (R2.1), RN1.2 (R2.1), RN1.2 (R2.1), RN1.2 (R2.1), RN1.2 (R2.1), RN1.2 (R2.1), RN1.2 (R2.1), RN1.2 (R2.1), RN1.2 (R2.1), RN1.2 (R2.1), RN1.2 (R2.1), RN1.3 (R3.1), RN1.3 (R3.1), RN1.3 (R3.1), RN1.3 (R3.1), RN1.3 (R3.1), RN1.3 (R3.1), RN1.3 (R3.1), RN1.3 (R3.1), RN1.3 (R3.1), RN1.3 (R3.1), RN1.3 (R3.1), RN1.3 (R3.1), RN1.4 (R4.1), RN1.4 (R4.1), RN1.4 (R4.1), RN1.4 (R4.1), RN1.4 (R4.1), RN1.4 (R4.1), RN1.4 (R4.1), RN1.4 (R4.1), RN1.4 (R4.1), RN1.4 (R4.1), RN1.4 (R4.1), RN1.4 (R4.1)
- net 040A0: now also RN1.6 (R3.2)
- net 040A1: now also RN1.5 (R4.2)
- net 040A2: now also RN1.8 (R1.2)
- net 040A3: now also RN1.7 (R2.2)
- net D040_0: now also RN1.8 (R1.2)
- net D040_1: now also RN1.7 (R2.2)
- net D040_10: now also RN1.7 (R2.2)
- net D040_11: now also RN1.8 (R1.2)
- net D040_12: now also RN1.5 (R4.2)
- net D040_13: now also RN1.6 (R3.2)
- net D040_14: now also RN1.7 (R2.2)
- net D040_15: now also RN1.8 (R1.2)
- net D040_16: now also RN1.5 (R4.2)
- net D040_17: now also RN1.6 (R3.2)
- net D040_18: now also RN1.7 (R2.2)
- net D040_19: now also RN1.8 (R1.2)
- net D040_2: now also RN1.6 (R3.2)
- net D040_20: now also RN1.5 (R4.2)
- net D040_21: now also RN1.6 (R3.2)
- net D040_22: now also RN1.7 (R2.2)
- net D040_23: now also RN1.8 (R1.2)
- net D040_24: now also RN1.8 (R1.2)
- net D040_25: now also RN1.7 (R2.2)
- net D040_26: now also RN1.6 (R3.2)
- net D040_27: now also RN1.5 (R4.2)
- net D040_28: now also RN1.8 (R1.2)
- net D040_29: now also RN1.7 (R2.2)
- net D040_3: now also RN1.5 (R4.2)
- net D040_30: now also RN1.6 (R3.2)
- net D040_31: now also RN1.5 (R4.2)
- net D040_4: now also RN1.8 (R1.2)
- net D040_5: now also RN1.7 (R2.2)
- net D040_6: now also RN1.6 (R3.2)
- net D040_7: now also RN1.5 (R4.2)
- net D040_8: now also RN1.5 (R4.2)
- net D040_9: now also RN1.6 (R3.2)
- net R_W040: now also RN1.7 (R2.2)
- net SIZ40_0: now also RN1.5 (R4.2)
- net SIZ40_1: now also RN1.6 (R3.2)
- net TM0: now also RN1.6 (R3.2)
- net TM1: now also RN1.5 (R4.2)
- net TM2: now also RN1.8 (R1.2)
- net TT0: now also RN1.7 (R2.2)
- net TT1: now also RN1.8 (R1.2)
- net _LOCK: now also RN1.6 (R3.2)
- net _LOCKE: now also RN1.5 (R4.2)
- net _TA: now also RN1.7 (R2.2)
- net _TEA: now also RN1.8 (R1.2)
